File: hw-tester/v0/memory-tester.kicad_sch (KiCad schematic)
At the start: 7 parts, among them J1 Conn_01x08, J2 Conn_02x14_Odd_Even, U2 74HCT595, U3 74HCT595, U4 74HCT595, U5 74HCT595, U6 74LS597

Commit message: Cleaned up a HW bug in the tester, provided docs
Connections:
- net A15: no longer U5.14 (SER)
- net A7: no longer U2.14 (SER)
- net C7: no longer U3.14 (SER)
- net CHAIN2: now reaches U2.9 (QH')
- net CHAIN2: now also U5.14 (SER)
- net CHAIN1: now reaches U3.9 (QH')
- net CHAIN1: now also U2.14 (SER)
- net CHAIN0: now reaches U4.9 (QH')
- net CHAIN0: now also U3.14 (SER)
- no-connect marks 9 -> 6
Other:
- company: (none) -> Bruce MacKinnon - KC1FSZ
- title: (none) -> Memory Tester
